File: Nucleo8x8Shield.kicad_pcb (KiCad board)
At the start: 2 copper layers, 72 x 66.5 mm, 95 parts, among them Q1 BSS138, Q2 BSS138, Q3 BSS138, Q4 BSS138, Q5 BSS138, Q6 BSS138, Q7 BSS138, Q8 BSS138, SW1 BTN1, SW2 BTN2, U1 NUCLEO-L432KC

Commit message: Fix LED reference designators overwritten by matrix coordinate labels
Six LED footprints (D1, D2, D3, D9, D63, D64) had their Reference
field overwritten with matrix coordinate text (0,0 / 0,1 / 0,2 /
1,0 / 7,6 / 7,7) instead of the actual designator, breaking the
schematic-to-layout reference match.

Restore the correct D-designators (hidden, as on every other LED)
and add the coordinate labels back as separate silkscreen text
items at the same position, so the board still shows the matrix
addressing hints without corrupting the footprint references.
Parts:
- renumbered 0,0 to D1, 0,1 to D2, 0,2 to D3, 7,6 to D63, 7,7 to D64, 1,0 to D9
Changed lines of the file:
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@@
 		(descr "LED SMD 0805 (2012 Metric), square (rectangular) end terminal, IPC-7351 nominal, (Body size source: https://docs.google.com/spreadsheets/d/1BsfQQcO9C6DZCsRaXUlFlo91Tg2WpOkGARC1WS5S8t0/edit?usp=sharing), generated with kicad-footprint-generator")
 		(tags "LED handsolder")
-		(property "Reference" "7,7"
+		(property "Reference" "D64"
 			(at -3.055 0 0)
 			(layer "F.SilkS")
+			(hide yes)
 			(effects
 				(font
@@
 			(layer "F.Fab")
 		)
+		(fp_text user "7,7"
+			(at -3.055 0 0)
+			(layer "F.SilkS")
+			(effects
+				(font
+					(size 1 1)
+					(thickness 0.15)
+				)
+			)
+		)
 		(fp_text user "${REFERENCE}"
 			(at 0 0 90)
@@
 		(descr "LED SMD 0805 (2012 Metric), square (rectangular) end terminal, IPC-7351 nominal, (Body size source: https://docs.google.com/spreadsheets/d/1BsfQQcO9C6DZCsRaXUlFlo91Tg2WpOkGARC1WS5S8t0/edit?usp=sharing), generated with kicad-footprint-generator")
 		(tags "LED handsolder")
-		(property "Reference" "0,2"
+		(property "Reference" "D3"
 			(at 2.945 0 180)
 			(layer "F.SilkS")
+			(hide yes)
 			(effects
 				(font
@@
 			(layer "F.Fab")
 		)
+		(fp_text user "0,2"
+			(at 2.945 0 180)
+			(layer "F.SilkS")
+			(effects
+				(font
+					(size 1 1)
+					(thickness 0.15)
+				)
+			)
+		)
 		(fp_text user "${REFERENCE}"
 			(at 0 0 90)
@@
 		(descr "LED SMD 0805 (2012 Metric), square (rectangular) end terminal, IPC-7351 nominal, (Body size source: https://docs.google.com/spreadsheets/d/1BsfQQcO9C6DZCsRaXUlFlo91Tg2WpOkGARC1WS5S8t0/edit?usp=sharing), generated with kicad-footprint-generator")
 		(tags "LED handsolder")
-		(property "Reference" "0,0"
+		(property "Reference" "D1"
 			(at 2.945 0 180)
 			(layer "F.SilkS")
+			(hide yes)
 			(effects
 				(font
@@
 			(layer "F.Fab")
 		)
+		(fp_text user "0,0"
+			(at 2.945 0 180)
+			(layer "F.SilkS")
+			(effects
+				(font
+					(size 1 1)
+					(thickness 0.15)
+				)
+			)
+		)
 		(fp_text user "${REFERENCE}"
 			(at 0 0 90)
@@
 		(descr "LED SMD 0805 (2012 Metric), square (rectangular) end terminal, IPC-7351 nominal, (Body size source: https://docs.google.com/spreadsheets/d/1BsfQQcO9C6DZCsRaXUlFlo91Tg2WpOkGARC1WS5S8t0/edit?usp=sharing), generated with kicad-footprint-generator")
 		(tags "LED handsolder")
-		(property "Reference" "1,0"
+		(property "Reference" "D9"
 			(at -0.055 -2.5 180)
 			(layer "F.SilkS")
@@
 		(descr "LED SMD 0805 (2012 Metric), square (rectangular) end terminal, IPC-7351 nominal, (Body size source: https://docs.google.com/spreadsheets/d/1BsfQQcO9C6DZCsRaXUlFlo91Tg2WpOkGARC1WS5S8t0/edit?usp=sharing), generated with kicad-footprint-generator")
 		(tags "LED handsolder")
-		(property "Reference" "7,6"
+		(property "Reference" "D63"
 			(at -3.055 0 180)
 			(layer "F.SilkS")
+			(hide yes)
 			(effects
 				(font
@@
 			(layer "F.Fab")
 		)
+		(fp_text user "7,6"
+			(at -3.055 0 180)
+			(layer "F.SilkS")
+			(effects
+				(font
+					(size 1 1)
+					(thickness 0.15)
+				)
+			)
+		)
 		(fp_text user "${REFERENCE}"
 			(at 0 0 90)
@@
 		(descr "LED SMD 0805 (2012 Metric), square (rectangular) end terminal, IPC-7351 nominal, (Body size source: https://docs.google.com/spreadsheets/d/1BsfQQcO9C6DZCsRaXUlFlo91Tg2WpOkGARC1WS5S8t0/edit?usp=sharing), generated with kicad-footprint-generator")
 		(tags "LED handsolder")
-		(property "Reference" "0,1"
+		(property "Reference" "D2"
 			(at 2.945 0 180)
 			(layer "F.SilkS")
+			(hide yes)
 			(effects
 				(font
@@
 			(layer "F.Fab")
 		)
+		(fp_text user "0,1"
+			(at 2.945 0 180)
+			(layer "F.SilkS")
+			(effects
+				(font
+					(size 1 1)
+					(thickness 0.15)
+				)
+			)
+		)
 		(fp_text user "${REFERENCE}"
